File: Hardware/Basic/Top/HolmesAndWatchson-BASIC-TOP.sch (EAGLE design)
At the start: 51 parts, among them SW1 SWITCH.MOM, SW2 SWITCH.MOM, U2 NRF52832_MODULE_MDBT42, U4 PCF8523

Commit message: Take002 and top board schematic complete
Parts:
- removed C2: 1u, LinnesLab-Passives:CAPACITOR0603
- removed R8, R9: 10k, LinnesLab-Passives:RESISTOR0603
- removed SD2: (no value), LinnesLab-Connectors:MICROSD
- removed U4: PCF8523, LinnesLab-Clocks:PCF8523
- removed XTAL3: 32.7680kHz, LinnesLab-Clocks:CRYSTALECS-.327-12.5-12-C-TR
- added C22: 100n, LinnesLab-Passives:CAPACITOR0603
- added C23, C24: 47p, LinnesLab-Passives:CAPACITOR0603
- added J1: (no value), LinnesLab-Connectors:CONN_061.27MM
- added JP2: (no value), LinnesLab-Switches:JUMPER-SMT_2_NO_SILK
- added LED5: RED, LinnesLab-LED:LED0603
- added LED6: YELLOW, LinnesLab-LED:LED0603
- added R1, R2: 0, LinnesLab-Passives:RESISTOR0603
- added R17, R18: 27, LinnesLab-Passives:RESISTOR0603
- added R19, R20: 1k, LinnesLab-Passives:RESISTOR0603
- added U5: FT231XS, LinnesLab-DigitalIC:FT231XS
Connections:
- removed net BATT: R13.1, R14.2
- removed net CD1: SD2.CARD_DETECT
- removed net CD2: SD2.CARD_DETECT1
- removed net CHRG.STAT: CHRG2.STAT, R12.1
- removed net CS.OLED: U3./CS
- removed net DC.OLED: U3.DC/I2C_SA0
- removed net N$19: U4.OSCO, XTAL3.1
- removed net N$20: U4.OSCI, XTAL3.2
- removed net RESET.OLED: U3./RES
- removed net RXD: U2.P0.08
- removed net SD.CS: SD2.CS
- removed net SW1: SW1.1, SW2.1
- removed net TXD: U2.P0.06
- removed net VBATT: U4.VBAT
- new net !CTS: JP2.2, U5.!CTS
- new net A4/BATT: R13.1, R14.2, U2.P0.28/AIN4
- new net A6/TIA: U2.P0.30/AIN6
- new net A7/PPG: U2.P0.31/AIN7
- new net D11/SW1: SW1.1, U2.P0.11
- new net D15/SW2: SW2.1, U2.P0.15
- new net D16/CS.OLED: U2.P0.16, U3./CS
- new net D27/CHRG.STATUS: CHRG2.STAT, R12.1, U2.P0.27
- new net D29/LED.CTRL: U2.P0.29/AIN5
- new net D3/RESET.OLED: U2.P0.03/AIN1, U3./RES
- new net D4/DC.OLED: U2.P0.04/AIN2, U3.DC/I2C_SA0
- new net FT3V3: U5.3V3OUT
- new net N$23: R17.2, U5.USBDM
- new net N$24: R18.2, U5.USBDP
- new net N$25: LED5.C, R19.2
- new net N$26: LED6.C, R20.2
- new net RXD.FT: R2.1, U5.RXD
- new net RXD.NRF: R1.2, U2.P0.08
- new net RXLED: R19.1, U5.CBUS1
- new net TXD.FT: R1.1, U5.TXD
- new net TXD.NRF: R2.2, U2.P0.06
- new net TXLED: R20.1, U5.CBUS2
- net 3.3V: now also C22.2, LED5.A, LED6.A, U5.!RESET, U5.VCCIO; no longer C2.1, R8.2, R9.2, SD2.VDD, U4.VDD
- net DTR: now also U5.!DTR
- net GND: now also C22.1, C23.2, C24.1, JP2.1, U5.GND@16, U5.GND@6; no longer C2.2, SD2.GND, SD2.GND1, SD2.VSS, U4.VSS
- net MISO: no longer SD2.DATA_OUT
- net MOSI: no longer SD2.DATA_IN
- net SCK: no longer SD2.SCLK
- net SCL: no longer R8.1, U4.SCL
- net SDA: no longer R9.1, U4.SDA
- net USB+: now also C23.1, R18.1
- net USB-: now also C24.2, R17.1
- net V_USB: now also U5.VCC
Other:
- note added: "I don't remember if CTS needs to be grounded or left floating so here's a jumper to ground so it can be configued either way dynamically."
- note added: "TXD goes to RX on the other device RXD goes to TX on the other device"
- note removed: "Back-up battery if desired"
- note removed: "Connect MISO, MOSI, and SCK to appropriate pins on microcontroller. Those are SPI pins and are generally prespecified. You have more flexibility with the SD.CS pin."
- note removed: "I2C Address = 0x68h"
- note removed: "REAL-TIME CLOCK"
- note removed: "RTC"
- note removed: "SD CARD"
- moved on the sheet: C10, C11, C8, C9, R6, SW1, SW4, XTAL2

Commit message: middle of take004 - routing TOP board
Other:
- note added: "FTDI SERIAL-TO-USB CONVERTER"
- moved on the sheet: C22, C23, C24, JP2, LED5, LED6, R1, R17, R18, R19, R2, R20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

Commit message: OLED routing
Parts:
- removed C10, C11: 300p, LinnesLab-Passives:CAPACITOR0603
Connections:
- net GND: no longer C10.2, C11.2
- net P0.09/NFC1: no longer C11.1
- net P0.10/NFC2: no longer C10.1
Changed lines of the file:
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@@
 <part name="GND15" library="LinnesLab-Symbols" deviceset="GND" device=""/>
 <part name="GND16" library="LinnesLab-Symbols" deviceset="GND" device=""/>
-<part name="GND17" library="LinnesLab-Symbols" deviceset="GND" device=""/>
-<part name="GND18" library="LinnesLab-Symbols" deviceset="GND" device=""/>
 <part name="GND19" library="LinnesLab-Symbols" deviceset="GND" device=""/>
 <part name="GND20" library="LinnesLab-Symbols" deviceset="GND" device=""/>
@@
 <part name="C8" library="LinnesLab-Passives" deviceset="CAPACITOR" device="0603" package3d_urn="urn:adsk.eagle:package:15661989/2"/>
 <part name="C9" library="LinnesLab-Passives" deviceset="CAPACITOR" device="0603" package3d_urn="urn:adsk.eagle:package:15661989/2"/>
-<part name="C10" library="LinnesLab-Passives" deviceset="CAPACITOR" device="0603" package3d_urn="urn:adsk.eagle:package:15661989/2" value="300p"/>
-<part name="C11" library="LinnesLab-Passives" deviceset="CAPACITOR" device="0603" package3d_urn="urn:adsk.eagle:package:15661989/2" value="300p"/>
 <part name="C12" library="LinnesLab-Passives" deviceset="CAPACITOR" device="0805" package3d_urn="urn:adsk.eagle:package:15662010/2" value="10u"/>
 <part name="L2" library="LinnesLab-Passives" deviceset="INDUCTOR" device="0603" override_package3d_urn="urn:adsk.eagle:package:18592195/2" override_package_urn="urn:adsk.eagle:footprint:18592196/1" value="10u"/>
@@
 <attribute name="VALUE" x="154.94" y="406.146" size="1.778" layer="96" align="top-center"/>
 </instance>
-<instance part="GND17" gate="G$1" x="157.48" y="370.84" smashed="yes">
-<attribute name="VALUE" x="157.48" y="370.586" size="1.778" layer="96" align="top-center"/>
-</instance>
-<instance part="GND18" gate="G$1" x="144.78" y="370.84" smashed="yes">
-<attribute name="VALUE" x="144.78" y="370.586" size="1.778" layer="96" align="top-center"/>
-</instance>
 <instance part="GND19" gate="G$1" x="134.62" y="370.84" smashed="yes">
 <attribute name="VALUE" x="134.62" y="370.586" size="1.778" layer="96" align="top-center"/>
@@
 <attribute name="NAME" x="136.144" y="381.381" size="1.778" layer="95"/>
 <attribute name="VALUE" x="136.144" y="376.301" size="1.778" layer="96"/>
-</instance>
-<instance part="C10" gate="G$1" x="157.48" y="378.46" smashed="yes">
-<attribute name="NAME" x="159.004" y="381.381" size="1.778" layer="95"/>
-<attribute name="VALUE" x="159.004" y="376.301" size="1.778" layer="96"/>
-</instance>
-<instance part="C11" gate="G$1" x="144.78" y="378.46" smashed="yes">
-<attribute name="NAME" x="146.304" y="381.381" size="1.778" layer="95"/>
-<attribute name="VALUE" x="146.304" y="376.301" size="1.778" layer="96"/>
 </instance>
 <instance part="C12" gate="G$1" x="114.3" y="419.1" smashed="yes" rot="R180">
@@
 <pinref part="GND20" gate="G$1" pin="GND"/>
 <pinref part="C8" gate="G$1" pin="1"/>
-</segment>
-<segment>
-<pinref part="C11" gate="G$1" pin="2"/>
-<pinref part="GND18" gate="G$1" pin="GND"/>
-<wire x1="144.78" y1="373.38" x2="144.78" y2="375.92" width="0.1524" layer="91"/>
-</segment>
-<segment>
-<pinref part="C10" gate="G$1" pin="2"/>
-<pinref part="GND17" gate="G$1" pin="GND"/>
-<wire x1="157.48" y1="373.38" x2="157.48" y2="375.92" width="0.1524" layer="91"/>
 </segment>
 <segment>
@@
 <wire x1="144.78" y1="386.08" x2="149.86" y2="386.08" width="0.1524" layer="91"/>
 <wire x1="144.78" y1="386.08" x2="144.78" y2="383.54" width="0.1524" layer="91"/>
-<pinref part="C11" gate="G$1" pin="1"/>
 <pinref part="U2" gate="G$1" pin="P0.09"/>
 <label x="149.86" y="388.62" size="1.27" layer="95" rot="R180" xref="yes"/>
@@
 <wire x1="152.4" y1="386.08" x2="157.48" y2="386.08" width="0.1524" layer="91"/>
 <wire x1="157.48" y1="386.08" x2="157.48" y2="383.54" width="0.1524" layer="91"/>
-<pinref part="C10" gate="G$1" pin="1"/>
 <pinref part="U2" gate="G$1" pin="P0.10"/>
 <label x="152.4" y="388.62" size="1.27" layer="95" xref="yes"/>

Commit message: continue editing top board
Parts:
- removed R15: 100k, LinnesLab-Passives:RESISTOR0603
Connections:
- net 3.3V: no longer R15.2
- net GND: no longer R15.1
Changed lines of the file:
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@@
 <part name="SUPPLY16" library="LinnesLab-Symbols" deviceset="VLIPO" device=""/>
 <part name="GND43" library="LinnesLab-Symbols" deviceset="GND" device=""/>
-<part name="R15" library="LinnesLab-Passives" deviceset="RESISTOR" device="0603" package3d_urn="urn:adsk.eagle:package:15661944/2" value="100k"/>
-<part name="GND44" library="LinnesLab-Symbols" deviceset="GND" device=""/>
 <part name="SUPPLY17" library="LinnesLab-Symbols" deviceset="VIN" device=""/>
 <part name="SW1" library="LinnesLab-Switches" deviceset="SWITCH.MOM" device=""/>
@@
 <attribute name="VALUE" x="162.56" y="246.126" size="1.778" layer="96" align="top-center"/>
 </instance>
-<instance part="R15" gate="G$1" x="175.26" y="281.94" smashed="yes" rot="R90">
-<attribute name="NAME" x="173.7614" y="278.13" size="1.778" layer="95" rot="R90"/>
-<attribute name="VALUE" x="178.562" y="278.13" size="1.778" layer="96" rot="R90"/>
-</instance>
-<instance part="GND44" gate="G$1" x="175.26" y="271.78" smashed="yes">
-<attribute name="VALUE" x="175.26" y="271.526" size="1.778" layer="96" align="top-center"/>
-</instance>
 <instance part="SUPPLY17" gate="G$1" x="116.84" y="292.1" smashed="yes">
 <attribute name="VALUE" x="116.84" y="294.894" size="1.778" layer="96" align="bottom-center"/>
@@
 </segment>
 <segment>
-<pinref part="R15" gate="G$1" pin="1"/>
-<pinref part="GND44" gate="G$1" pin="GND"/>
-<wire x1="175.26" y1="274.32" x2="175.26" y2="276.86" width="0.1524" layer="91"/>
-</segment>
-<segment>
 <pinref part="SW1" gate="G$1" pin="3"/>
 <wire x1="515.62" y1="327.66" x2="518.16" y2="327.66" width="0.1524" layer="91" style="longdash"/>
@@
 <wire x1="165.1" y1="292.1" x2="165.1" y2="289.56" width="0.1524" layer="91"/>
 <junction x="165.1" y="289.56"/>
-<wire x1="165.1" y1="289.56" x2="175.26" y2="289.56" width="0.1524" layer="91"/>
-<pinref part="R15" gate="G$1" pin="2"/>
-<wire x1="175.26" y1="289.56" x2="175.26" y2="287.02" width="0.1524" layer="91"/>
-</segment>
-<segment>
+</segment>
+<segment>
