File: Hardware/Basic/Top/HolmesAndWatchson-BASIC-TOP.brd (EAGLE design)
At the start: 0 parts

Commit message: top board rev1
Parts:
- added C10, C11: 300p, LinnesLab-Passives:C0603
- added C12: 10u, LinnesLab-Passives:C0805
- added C13, C15, C17, C18, C19: 2.2uF, LinnesLab-Passives:C0402
- added C14: 100n, LinnesLab-Passives:C0603
- added C16: 10uF, LinnesLab-Passives:C0603
- added C2, C5, C6, C7: 1u, LinnesLab-Passives:C0603
- added C20, C21: 4.7u, LinnesLab-Passives:C0603
- added C8, C9: (no value), LinnesLab-Passives:C0603
- added CHRG2: MCP73831, LinnesLab-Power:SOT23-5
- added CORTEX1: CORTEX_DEBUG_PTH, LinnesLab-Connectors:2X5-PTH-1.27MM
- added D1, D4, D5: (no value), LinnesLab-DiscreteSemi:USC
- added J2: (no value), LinnesLab-Connectors:1X02
- added L2: 10u, LinnesLab-Passives:L0603
- added LDO2: MIC5504, LinnesLab-Power:SOT23-5
- added LED3: RED, LinnesLab-LED:LED-0603
- added LED4: BLUE, LinnesLab-LED:LED-0603
- added R11: (no value), LinnesLab-Passives:R0603
- added R12, R13, R14, R15: 100k, LinnesLab-Passives:R0603
- added R3, R4: 1k, LinnesLab-Passives:R0603
- added R5, R6, R8, R9: 10k, LinnesLab-Passives:R0603
- added R7: 390k, LinnesLab-Passives:R0603
- added SD2: (no value), LinnesLab-Connectors:MICROSD
- added SW1, SW2: SWITCH.MOM, LinnesLab-Switches:TACTILE_SWITCH_SMD_6.2MM_TALL
- added SW3, SW4: (no value), LinnesLab-Switches:BUTTON-GULLWING
- added U2: NRF52832_MODULE_MDBT42, LinnesLab-Microcontrollers:BLE_MODULE_RAYTAC_MDBT42
- added U3: (no value), LinnesLab-Displays:UG-2864HSWEG01_0.96IN_NO-WRAPAROUND
- added U4: PCF8523, LinnesLab-Clocks:SO8
- added USB2: USB.MICRO-BIGGERPADS, LinnesLab-Connectors:USB-MICRO-01.BIGGERPADS
- added XTAL2: 32.768kHz, LinnesLab-Clocks:2-SMD.NOLEAD.2.0MMTO1.2MM
- added XTAL3: 32.7680kHz, LinnesLab-Clocks:2-SMD.NOLEAD.2.0MMTO1.2MM
Connections:
- new net 3.3V: C12.2, C17.2, C19.2, C2.1, C6.1, CORTEX1.1, D1.-, LDO2.5, R15.2, R5.2, R8.2, R9.2, SD2.4, U2.11, U3.6, U3.9, U4.8
- new net BATT: R13.1, R14.2
- new net CD1: SD2.CD1
- new net CD2: SD2.CD2
- new net CHRG.STAT: CHRG2.1, R12.1
- new net CS.OLED: U3.13
- new net DC.OLED: U3.15
- new net DFU: SW3.3, U2.34
- new net DTR: C14.1
- new net FRST: U2.38
- new net GND: C10.2, C11.2, C12.1, C16.1, C17.1, C18.1, C19.1, C2.2, C20.2, C21.1, C5.1, C6.2, C7.2, C8.1, C9.2, CHRG2.2, CORTEX1.3, CORTEX1.5, CORTEX1.7, CORTEX1.9, J2.1, LDO2.2, LED3.C, LED4.C, R11.1, R14.1, R15.1, R6.1, R7.2, SD2.6, SD2.MT1, SD2.MT2, SW1.B1, SW1.B2, SW2.B1, SW2.B2, SW3.1, SW4.3, U2.1, U2.12, U2.24, U2.39, U3.1, U3.10, U3.12, U3.29, U3.30, U3.8, U4.4, USB2.5, USB2.S1, USB2.S2, USB2.S3, USB2.S4, USB2.S5, USB2.S6
- new net LED1: R3.2, U2.31
- new net LED2: R4.2, U2.33
- new net MISO: SD2.7, U2.28
- new net MOSI: SD2.3, U2.27, U3.19
- new net N$1: R6.2, U3.11
- new net N$10: LED4.A, R4.1
- new net N$11: L2.1, U2.10
- new net N$12: C7.1, L2.2, U2.9
- new net N$13: C16.2, U3.28
- new net N$14: CORTEX1.8
- new net N$15: C18.2, U3.27
- new net N$17: CHRG2.5, R11.2
- new net N$19: U4.2, XTAL3.P$1
- new net N$2: R7.1, U3.26
- new net N$20: U4.1, XTAL3.P$2
- new net N$3: C13.2, U3.2
- new net N$4: C8.2, U2.13, XTAL2.P$1
- new net N$5: C13.1, U3.3
- new net N$6: C9.1, U2.14, XTAL2.P$2
- new net N$7: C15.2, U3.4
- new net N$8: C15.1, U3.5
- new net N$9: LED3.A, R3.1
- new net P0.09/NFC1: C11.1, U2.22
- new net P0.10/NFC2: C10.1, U2.23
- new net RESET: C14.2, CORTEX1.10, D1.+, R5.1, SW4.1, U2.35
- new net RESET.OLED: U3.14
- new net RXD: U2.21
- new net SCK: SD2.5, U2.26, U3.18
- new net SCL: R8.1, U2.3, U4.6
- new net SD.CS: SD2.2
- new net SDA: R9.1, U2.2, U4.5
- new net SW1: SW1.A1, SW2.A1
- new net SWCLK: CORTEX1.4, U2.36
- new net SWDIO: CORTEX1.2, U2.37
- new net SWO: CORTEX1.6, U2.32
- new net TXD: U2.19
- new net USB+: USB2.3
- new net USB-: USB2.2
- new net VBATT: U4.3
- new net VIN: C21.2, C5.2, CHRG2.4, D4.-, D5.-, LDO2.1, LDO2.3, R12.2
- new net VLIPO: C20.1, CHRG2.3, D4.+, J2.2, R13.2
- new net V_USB: D5.+, USB2.1
Other:
- board outline added: 38 x 38 mm

Commit message: Take002 and top board schematic complete
Parts:
- removed C2: 1u, LinnesLab-Passives:C0603
- removed R8, R9: 10k, LinnesLab-Passives:R0603
- removed SD2: (no value), LinnesLab-Connectors:MICROSD
- removed U4: PCF8523, LinnesLab-Clocks:SO8
- removed XTAL3: 32.7680kHz, LinnesLab-Clocks:2-SMD.NOLEAD.2.0MMTO1.2MM
- added C22: 100n, LinnesLab-Passives:C0603
- added C23, C24: 47p, LinnesLab-Passives:C0603
- added J1: (no value), LinnesLab-Connectors:1X06_1.27MM
- added JP2: (no value), LinnesLab-Switches:SMT-JUMPER_2_NO_SILK
- added LED5: RED, LinnesLab-LED:LED-0603
- added LED6: YELLOW, LinnesLab-LED:LED-0603
- added R1, R2: 0, LinnesLab-Passives:R0603
- added R17, R18: 27, LinnesLab-Passives:R0603
- added R19, R20: 1k, LinnesLab-Passives:R0603
- added U5: FT231XS, LinnesLab-DigitalIC:SSOP20_L
- moved SW3 33.9 mm to (14.7, 29.2)
- moved R5 24.6 mm to (21.6, 12.2), turned to 180 degrees
- moved D1 23.1 mm to (25.5, 12.1), turned to 180 degrees
- moved C14 22.9 mm to (28.6, 11.2)
- moved LED4 21.1 mm to (32.0, 9.40)
- moved CORTEX1 15.9 mm to (33.9, 16.9)
- moved R3 15.5 mm to (31.8, 11.7), turned to 0 degrees
- moved R4 15.2 mm to (32.3, 14.0)
- moved LED3 14.1 mm to (36.1, 12.7), turned to 90 degrees
- moved C12 14.0 mm to (9.27, 31.8)
- moved C10 11.0 mm to (11.8, 29.1), turned to 90 degrees
- moved C7 10.5 mm to (8.76, 29.5), turned to 0 degrees
- moved C11 10.5 mm to (13.5, 32.3)
- moved SW4 7.73 mm to (16.1, 24.1)
- moved C19 7.62 mm to (9.09, 27.9)
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Connections:
- removed net BATT: R13.1, R14.2
- removed net CD1: SD2.CD1
- removed net CD2: SD2.CD2
- removed net CHRG.STAT: CHRG2.1, R12.1
- removed net CS.OLED: U3.13
- removed net DC.OLED: U3.15
- removed net N$19: U4.2, XTAL3.P$1
- removed net N$20: U4.1, XTAL3.P$2
- removed net RESET.OLED: U3.14
- removed net RXD: U2.21
- removed net SD.CS: SD2.2
- removed net SW1: SW1.A1, SW2.A1
- removed net TXD: U2.19
- removed net VBATT: U4.3
- new net !CTS: JP2.2, U5.9
- new net A4/BATT: R13.1, R14.2, U2.5
- new net A6/TIA: U2.7
- new net A7/PPG: U2.8
- new net D11/SW1: SW1.A1, U2.25
- new net D15/SW2: SW2.A1, U2.29
- new net D16/CS.OLED: U2.30, U3.13
- new net D27/CHRG.STATUS: CHRG2.1, R12.1, U2.4
- new net D29/LED.CTRL: U2.6
- new net D3/RESET.OLED: U2.16, U3.14
- new net D4/DC.OLED: U2.17, U3.15
- new net FT3V3: U5.13
- new net N$23: R17.2, U5.12
- new net N$24: R18.2, U5.11
- new net N$25: LED5.C, R19.2
- new net N$26: LED6.C, R20.2
- new net RXD.FT: R2.1, U5.4
- new net RXD.NRF: R1.2, U2.21
- new net RXLED: R19.1, U5.17
- new net TXD.FT: R1.1, U5.20
- new net TXD.NRF: R2.2, U2.19
- new net TXLED: R20.1, U5.10
- net 3.3V: now also C22.2, LED5.A, LED6.A, U5.14, U5.3; no longer C2.1, R8.2, R9.2, SD2.4, U4.8
- net DTR: now also U5.1
- net GND: now also C22.1, C23.2, C24.1, JP2.1, U5.16, U5.6; no longer C2.2, SD2.6, SD2.MT1, SD2.MT2, U4.4
- net MISO: no longer SD2.7
- net MOSI: no longer SD2.3
- net SCK: no longer SD2.5
- net SCL: no longer R8.1, U4.6
- net SDA: no longer R9.1, U4.5
- net USB+: now also C23.1, R18.1
- net USB-: now also C24.2, R17.1
- net V_USB: now also U5.15

Commit message: middle of take004 - routing TOP board
Parts:
- moved C23 66.1 mm to (18.0, -29.0), turned to 270 degrees
- moved LED5 60.1 mm to (18.8, -23.5), turned to 180 degrees
- moved JP2 59.4 mm to (5.77, -26.7), turned to 0 degrees
- moved LED6 58.7 mm to (19.3, -20.7), turned to 180 degrees
- moved C22 58.7 mm to (6.47, -21.8), turned to 90 degrees
- moved R19 56.5 mm to (15.5, -23.5), turned to 0 degrees
- moved R18 54.5 mm to (15.6, -28.2), turned to 180 degrees
- moved U5 53.3 mm to (10.5, -24.5)
- moved C24 52.0 mm to (18.0, -25.8), turned to 270 degrees
- moved D5 50.6 mm to (35.2, 41.6)
- moved R20 50.2 mm to (15.8, -20.7), turned to 0 degrees
- moved R17 49.0 mm to (15.6, -26.7), turned to 180 degrees
- moved D4 45.2 mm to (31.4, 41.1)
- moved LDO2 43.5 mm to (3.71, 46.4)
- moved CHRG2 41.0 mm to (14.4, 48.4)
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Routing:
- net TXLED: track 0.00 -> 13.1 mm, vias 0 -> 2
- net RXD.FT: track 0.00 -> 6.88 mm
- net N$12: track 0.00 -> 4.70 mm
- net TXD.FT: track 0.00 -> 3.45 mm
- net N$24: track 0.00 -> 2.08 mm
- net N$11: track 0.00 -> 1.92 mm
- net N$26: track 0.00 -> 1.73 mm
- net GND: track 0.00 -> 1.69 mm, vias 0 -> 1
- net N$25: track 0.00 -> 1.67 mm
- net USB+: track 0.00 -> 1.59 mm
- net USB-: track 0.00 -> 1.58 mm
- net N$23: track 0.00 -> 1.50 mm
- net RXLED: track 0.00 -> 1.39 mm

Commit message: OLED routing
Parts:
- removed C10, C11: 300p, LinnesLab-Passives:C0603
- moved C22 32.9 mm to (3.48, 11.0)
- moved JP2 32.9 mm to (2.78, 6.05)
- moved R2 32.9 mm to (5.78, 14.6)
- moved R20 32.9 mm to (12.8, 12.0)
- moved C23 32.9 mm to (15.0, 3.69)
- moved C24 32.9 mm to (15.0, 6.89)
- moved LED5 32.9 mm to (15.9, 9.26)
- moved LED6 32.9 mm to (16.3, 12.0)
- moved R1 32.9 mm to (10.8, 14.5)
- moved R17 32.9 mm to (12.6, 6.04)
- moved R18 32.9 mm to (12.6, 4.53)
- moved R19 32.9 mm to (12.5, 9.22)
- moved U5 32.9 mm to (7.55, 8.27)
- moved C16 21.7 mm to (32.0, 19.6), turned to 180 degrees
- moved R7 21.0 mm to (32.0, 16.9)
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Connections:
- net GND: no longer C10.2, C11.2
- net P0.09/NFC1: no longer C11.1
- net P0.10/NFC2: no longer C10.1
Routing:
- net GND: track 1.69 -> 20.2 mm, vias 1 -> 13
- net N$2: track 0.00 -> 6.73 mm
- net N$13: track 0.00 -> 5.45 mm
- net N$5: track 0.00 -> 5.30 mm
- net N$8: track 0.00 -> 5.04 mm
- net N$15: track 0.00 -> 4.16 mm
- net N$3: track 0.00 -> 3.71 mm
- net N$1: track 0.00 -> 3.56 mm
- net N$7: track 0.00 -> 3.44 mm
- net N$11: track 1.92 -> 3.41 mm
- net N$12: track 4.70 -> 5.49 mm
- added copper zone on layer 1, net 3.3V
- added copper zone on layer 16, net GND

Commit message: continue editing top board
Parts:
- removed R15: 100k, LinnesLab-Passives:R0603
- moved CHRG2 65.8 mm to (22.8, -16.9)
- moved D5 47.6 mm to (6.68, 3.47), flipped to the bottom, turned to 270 degrees
- moved D4 44.1 mm to (8.40, 3.54), flipped to the bottom, turned to 270 degrees
- moved C20 44.0 mm to (27.4, -18.0)
- moved LDO2 44.0 mm to (12.8, 3.32), flipped to the bottom, turned to 90 degrees
- moved C21 42.4 mm to (26.1, -21.1)
- moved C6 32.6 mm to (15.2, 7.58), flipped to the bottom, turned to 90 degrees
- moved R11 31.2 mm to (30.3, -19.2), turned to 270 degrees
- moved C22 27.1 mm to (-2.90, -15.4)
- moved JP2 27.1 mm to (-3.60, -20.3)
- moved R1 27.1 mm to (4.46, -11.9)
- moved R17 27.1 mm to (6.20, -20.3)
- moved R18 27.1 mm to (6.19, -21.8)
- moved R2 27.1 mm to (-0.60, -11.8)
- moved R20 27.1 mm to (6.43, -14.4)
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Connections:
- net 3.3V: no longer R15.2
- net GND: no longer R15.1
Routing:
- net VLIPO: track 0.00 -> 13.6 mm
- net VIN: track 0.00 -> 5.11 mm
- net V_USB: track 0.00 -> 2.08 mm
- net N$26: track 1.73 -> 3.25 mm
- net USB-: track 1.58 -> 2.76 mm
- net USB+: track 1.59 -> 2.77 mm
- net N$25: track 1.67 -> 2.83 mm

Commit message: finished take 005
Parts:
- moved R4 55.1 mm to (9.43, 50.5)
- moved R3 50.9 mm to (9.20, 48.0), turned to 180 degrees
- moved C9 46.4 mm to (34.9, 19.0), turned to 0 degrees
- moved C8 44.8 mm to (32.1, 17.4), turned to 180 degrees
- moved R11 41.4 mm to (2.98, 11.9), flipped to the bottom, turned to 180 degrees
- moved R14 37.2 mm to (2.14, 20.1), turned to 90 degrees
- moved R5 35.1 mm to (2.82, 27.4)
- moved D1 34.9 mm to (3.09, 29.8)
- moved C20 34.5 mm to (9.78, 11.7), flipped to the bottom, turned to 0 degrees
- moved R13 32.0 mm to (4.21, 20.0), turned to 270 degrees
- moved C21 30.4 mm to (11.7, 5.65), flipped to the bottom
- moved R12 29.9 mm to (12.4, 8.02), flipped to the bottom, turned to 270 degrees
- moved CHRG2 28.5 mm to (9.75, 8.52), flipped to the bottom, turned to 180 degrees
- moved C24 26.8 mm to (16.2, 6.40)
- moved C23 26.7 mm to (14.7, 3.35), turned to 90 degrees
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Routing:
- net USB-: track 2.76 -> 23.5 mm, vias 0 -> 1
- net TXLED: track 13.1 -> 0.11 mm, vias 2 -> 0
- net USB+: track 2.77 -> 15.3 mm, vias 0 -> 1
- net VLIPO: track 13.6 -> 25.5 mm
- net GND: track 20.2 -> 30.4 mm, vias 13 -> 16
- net N$6: track 0.00 -> 7.80 mm
- net N$17: track 0.00 -> 7.22 mm
- net N$4: track 0.00 -> 7.16 mm
- net VIN: track 5.11 -> 12.3 mm
- net RXD.FT: track 6.81 -> 0.00 mm
- net N$2: track 6.73 -> 0.00 mm
- net N$13: track 5.45 -> 0.00 mm
- net 3.3V: track 0.00 -> 2.50 mm, vias 0 -> 1
- net A4/BATT: track 0.00 -> 2.10 mm
- net SWDIO: track 0.00 -> 1.44 mm, vias 0 -> 1
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